File: pcb_designs/eps/MCU.kicad_sch (KiCad schematic)
At the start: 11 parts

Commit message: first commits to 3D models - gotta start grinding the project again
Parts:
- added C?: 1u, symbol Device:C
- added FB?: FerriteBead, symbol Device:FerriteBead
Connections:
- net +3.3V: now also C?.1, FB?.2
- net +3.3VA: now also FB?.1
- net GND: now also C?.2
- net RESET: now reaches U?.7 (NRST)
