File: pcb_designs/eps/eps.kicad_sch (KiCad schematic)
At the start: 0 parts

Commit message: first commits to 3D models - gotta start grinding the project again
Other:
- sheet MCU ports: added RESET; removed none
Changed lines of the file:
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@@
+			)
+		)
+		(pin "RESET" input
+			(at 123.19 72.39 180)
+			(effects
+				(font
+					(size 1.27 1.27)
+				)
+				(justify left)
 			)
 		)
